File: core/pcb/rev1.0/apex-iii-core/apex-iii-core.sch (EAGLE design)
At the start: 67 parts, among them IC1 CA3240ED

Commit message: i2c resistors
Parts:
- added I2C_RES, I2C_RES1: 4K7, rcl:R-EU_R0603
Connections:
- net I2C_SCL: now also I2C_RES.2
- net I2C_SDA: now also I2C_RES1.2
- net VCC: now also I2C_RES.1, I2C_RES1.1
Other:
- moved on the sheet: C10, FTDI
Changed lines of the file:
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@@
 <part name="GND31" library="SparkFun" deviceset="GND" device=""/>
 <part name="JP6" library="apex" deviceset="APEXHAB-LOGO" device="_APEXHAB"/>
+<part name="I2C_RES" library="rcl" deviceset="R-EU_" device="R0603" value="4K7"/>
+<part name="I2C_RES1" library="rcl" deviceset="R-EU_" device="R0603" value="4K7"/>
+<part name="P+18" library="SparkFun" deviceset="VCC" device=""/>
+<part name="P+19" library="SparkFun" deviceset="VCC" device=""/>
 </parts>
 <sheets>
@@
 <attribute name="VALUE" x="126.619" y="197.104" size="1.778" layer="96" rot="R180"/>
 </instance>
-<instance part="FTDI" gate="G$1" x="264.16" y="228.6" smashed="yes" rot="R180">
-<attribute name="NAME" x="269.24" y="217.678" size="1.778" layer="95" rot="R180"/>
-<attribute name="VALUE" x="276.86" y="238.76" size="1.778" layer="96" rot="R180"/>
+<instance part="FTDI" gate="G$1" x="307.34" y="215.9" smashed="yes" rot="R180">
+<attribute name="NAME" x="312.42" y="204.978" size="1.778" layer="95" rot="R180"/>
+<attribute name="VALUE" x="320.04" y="226.06" size="1.778" layer="96" rot="R180"/>
 </instance>
 <instance part="ICSP" gate="G$1" x="289.56" y="165.1" smashed="yes">
@@
 </instance>
 <instance part="FRAME2" gate="G$1" x="0" y="0"/>
-<instance part="GND9" gate="1" x="254" y="220.98" rot="R270"/>
-<instance part="C10" gate="G$1" x="254" y="243.84"/>
+<instance part="GND9" gate="1" x="297.18" y="208.28" rot="R270"/>
+<instance part="C10" gate="G$1" x="297.18" y="231.14"/>
 <instance part="P+6" gate="1" x="274.32" y="167.64"/>
 <instance part="GND10" gate="1" x="274.32" y="160.02"/>
@@
 <instance part="GND31" gate="1" x="198.12" y="116.84" rot="R270"/>
 <instance part="JP6" gate="G$1" x="317.5" y="25.4"/>
+<instance part="I2C_RES" gate="G$1" x="256.54" y="228.6" rot="R270"/>
+<instance part="I2C_RES1" gate="G$1" x="238.76" y="233.68" rot="R270"/>
+<instance part="P+18" gate="1" x="256.54" y="236.22"/>
+<instance part="P+19" gate="1" x="238.76" y="241.3"/>
 </instances>
 <busses>
@@
 </segment>
 <segment>
-<wire x1="256.54" y1="220.98" x2="259.08" y2="220.98" width="0.1524" layer="91"/>
+<wire x1="299.72" y1="208.28" x2="302.26" y2="208.28" width="0.1524" layer="91"/>
 <pinref part="GND9" gate="1" pin="GND"/>
 <pinref part="FTDI" gate="G$1" pin="6"/>
@@
 <pinref part="I2C-3" gate="-1" pin="S"/>
 </segment>
+<segment>
+<pinref part="I2C_RES1" gate="G$1" pin="1"/>
+<pinref part="P+19" gate="1" pin="VCC"/>
+<wire x1="238.76" y1="241.3" x2="238.76" y2="238.76" width="0.1524" layer="91"/>
+</segment>
+<segment>
+<pinref part="P+18" gate="1" pin="VCC"/>
+<pinref part="I2C_RES" gate="G$1" pin="1"/>
+<wire x1="256.54" y1="236.22" x2="256.54" y2="233.68" width="0.1524" layer="91"/>
+</segment>
 </net>
 <net name="VBATT" class="0">
@@
 <net name="N$9" class="0">
 <segment>
-<wire x1="243.84" y1="231.14" x2="259.08" y2="231.14" width="0.1524" layer="91"/>
-<wire x1="243.84" y1="231.14" x2="243.84" y2="208.28" width="0.1524" layer="91"/>
+<wire x1="243.84" y1="218.44" x2="302.26" y2="218.44" width="0.1524" layer="91"/>
+<wire x1="243.84" y1="218.44" x2="243.84" y2="208.28" width="0.1524" layer="91"/>
 <wire x1="243.84" y1="208.28" x2="218.44" y2="208.28" width="0.1524" layer="91"/>
 <pinref part="ARDUINO-ATMEGA328" gate="1" pin="DIGITAL_1(TX)"/>
@@
 <net name="N$10" class="0">
 <segment>
-<wire x1="259.08" y1="228.6" x2="241.3" y2="228.6" width="0.1524" layer="91"/>
+<wire x1="302.26" y1="215.9" x2="241.3" y2="215.9" width="0.1524" layer="91"/>
 <wire x1="218.44" y1="210.82" x2="241.3" y2="210.82" width="0.1524" layer="91"/>
-<wire x1="241.3" y1="210.82" x2="241.3" y2="228.6" width="0.1524" layer="91"/>
+<wire x1="241.3" y1="210.82" x2="241.3" y2="215.9" width="0.1524" layer="91"/>
 <pinref part="FTDI" gate="G$1" pin="3"/>
 <pinref part="ARDUINO-ATMEGA328" gate="1" pin="DIGITAL_0(RX)"/>
@@
 </segment>
 <segment>
-<wire x1="254" y1="248.92" x2="254" y2="251.46" width="0.1524" layer="91"/>
-<label x="254" y="251.46" size="1.778" layer="95" xref="yes"/>
+<wire x1="297.18" y1="236.22" x2="297.18" y2="238.76" width="0.1524" layer="91"/>
+<label x="297.18" y="238.76" size="1.778" layer="95" xref="yes"/>
 <pinref part="C10" gate="G$1" pin="1"/>
 </segment>
@@
 <net name="N$4" class="0">
 <segment>
-<wire x1="259.08" y1="233.68" x2="254" y2="233.68" width="0.1524" layer="91"/>
-<wire x1="254" y1="233.68" x2="254" y2="241.3" width="0.1524" layer="91"/>
+<wire x1="302.26" y1="220.98" x2="297.18" y2="220.98" width="0.1524" layer="91"/>
+<wire x1="297.18" y1="220.98" x2="297.18" y2="228.6" width="0.1524" layer="91"/>
 <pinref part="FTDI" gate="G$1" pin="1"/>
 <pinref part="C10" gate="G$1" pin="2"/>
@@
 </segment>
 <segment>
-<wire x1="218.44" y1="223.52" x2="220.98" y2="223.52" width="0.1524" layer="91"/>
-<label x="220.98" y="223.52" size="1.27" layer="95" xref="yes"/>
+<label x="241.3" y="223.52" size="1.27" layer="95" xref="yes"/>
 <pinref part="ARDUINO-ATMEGA328" gate="1" pin="ANALOG_4"/>
+<pinref part="I2C_RES1" gate="G$1" pin="2"/>
+<wire x1="218.44" y1="223.52" x2="238.76" y2="223.52" width="0.1524" layer="91"/>
+<wire x1="238.76" y1="223.52" x2="241.3" y2="223.52" width="0.1524" layer="91"/>
+<wire x1="238.76" y1="228.6" x2="238.76" y2="223.52" width="0.1524" layer="91"/>
+<junction x="238.76" y="223.52"/>
 </segment>
 <segment>
@@
 </segment>
 <segment>
-<wire x1="218.44" y1="220.98" x2="220.98" y2="220.98" width="0.1524" layer="91"/>
-<label x="220.98" y="220.98" size="1.27" layer="95" xref="yes"/>
+<label x="261.62" y="220.98" size="1.27" layer="95" xref="yes"/>
 <pinref part="ARDUINO-ATMEGA328" gate="1" pin="ANALOG_5"/>
-</segment>
-<segment>
+<pinref part="I2C_RES" gate="G$1" pin="2"/>
+<wire x1="218.44" y1="220.98" x2="256.54" y2="220.98" width="0.1524" layer="91"/>
+<wire x1="256.54" y1="220.98" x2="261.62" y2="220.98" width="0.1524" layer="91"/>
+<wire x1="256.54" y1="223.52" x2="256.54" y2="220.98" width="0.1524" layer="91"/>
+<junction x="256.54" y="220.98"/>
+</segment>
+<segment>

Commit message: end of day commit - board very messy
Parts:
- removed 1WIRE_PULL_UP, CS_PULL_UP_RES: 4.7K, rcl:R-EU_R0603
- removed GPS_RES: 100K, rcl:R-EU_R0603
- removed I2C-3: I2C_3, apex:22-27-2041-04
- removed I2C_RES: 4K7, rcl:R-EU_R0603
- removed NTR2_RES: 22K, rcl:R-EU_R0603
- removed UP_RES3: 1K5, rcl:R-EU_R0603
- removed UP_RES6: 1K, rcl:R-EU_R0603
- removed UP_RES7: 10K, rcl:R-EU_R0603
- added 1WIRE, CS_PULL_UP, I2C_RES2: 4K7, apex:R-EU_R0805
- added GPS_RES3, UP_RES2: 1K, apex:R-EU_R0805
- added NTR2_RES4, UP_RES1: 10K, apex:R-EU_R0805
- added UP_RES4: 1K5, apex:R-EU_R0805
- BATT, BATT2, GPS_RES1, I2C_RES1, MISO_RES, NTR2_RES2, NTR2_RES3, RES_PWR, STATUS_RES: device rcl:R-EU_R0603 -> apex:R-EU_R0805
- GPS_RES2: value 1K -> 100K; device rcl:R-EU_R0603 -> apex:R-EU_R0805
- NTR2_RES1: value 10K -> 22K; device rcl:R-EU_R0603 -> apex:R-EU_R0805
- renumbered IC1 to UPL, TEMP to TEMPEXT, TEMPA to TEMPADD
Connections:
- removed net N$7: NTR2_RES.1, NTR2_RES2.2
- new net N$16: NTR2_RES1.2, NTR2_RES2.1
- net GND: now also NTR2_RES4.2, UP_RES2.2, UP_RES4.2; no longer I2C-3-4.S, NTR2_RES1.2, UP_RES3.1, UP_RES6.2
- net GPS_RX: now also GPS_RES3.1; no longer GPS_RES2.1
- net GPS_TX: now also GPS_RES2.2; no longer GPS_RES1.2
- net I2C_SCL: now also I2C_RES2.2; no longer I2C-3-2.S, I2C_RES.2
- net I2C_SDA: no longer I2C-3-3.S
- net N$11: now also CS_PULL_UP.2; no longer CS_PULL_UP_RES.1
- net N$12: now also NTR2_RES2.2, NTR2_RES3.2, NTR2_RES4.1; no longer NTR2_RES1.1, NTR2_RES2.1, NTR2_RES3.1
- net N$13: now also GPS_RES1.1; no longer GPS_RES.1
- net N$14: now also GPS_RES3.2; no longer GPS_RES2.2
- net N$20: now also UP_RES4.1; no longer UP_RES3.2
- net N$22: now also UP_RES1.2; no longer UP_RES7.2
- net N$23: now also UP_RES2.1; no longer UP_RES6.1
- net N$8: now also STATUS_RES.2; no longer STATUS_RES.1
- net RANDOM: now also UP_RES1.1; no longer UP_RES7.1
- net SCK: now also STATUS_RES.1; no longer STATUS_RES.2
- net TEMPERATURE: now also 1WIRE.1; no longer 1WIRE_PULL_UP.1
- net TX_0: now also NTR2_RES1.1; no longer NTR2_RES.2
- net TX_1: now also NTR2_RES3.1; no longer NTR2_RES3.2
- net VCC: now also 1WIRE.2, CS_PULL_UP.1, GPS_RES1.2, GPS_RES2.1, I2C_RES2.1; no longer 1WIRE_PULL_UP.2, CS_PULL_UP_RES.2, GPS_RES.2, GPS_RES1.1, I2C-3-1.S, I2C_RES.1
Other:
- moved on the sheet: GPS_RES1, GPS_RES2, I2C-1-1, I2C-1-2, I2C-1-3, I2C-1-4, I2C-2-1, I2C-2-2, I2C-2-3, I2C-2-4, NTR2_RES1, NTR2_RES2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

Commit message: pcb mainly finished
Parts:
- OPAMP: value CA3240ED -> MAX4477
- renumbered UPL to OPAMP
Changed lines of the file:
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@@
 <part name="GND26" library="SparkFun" deviceset="GND" device=""/>
 <part name="NTR2" library="apex" deviceset="NTR2" device=""/>
-<part name="UPL" library="linear" deviceset="CA3240E" device="D"/>
+<part name="OPAMP" library="linear" deviceset="CA3240E" device="D" value="MAX4477"/>
 <part name="UP_CAP1" library="SparkFun" deviceset="CAP" device="0805" value="47nF"/>
 <part name="GND27" library="SparkFun" deviceset="GND" device=""/>
@@
 <instance part="GND26" gate="1" x="27.94" y="41.91" rot="R270"/>
 <instance part="NTR2" gate="G$1" x="325.12" y="114.3"/>
-<instance part="UPL" gate="B" x="320.04" y="60.96" smashed="yes" rot="MR0">
+<instance part="OPAMP" gate="B" x="320.04" y="60.96" smashed="yes" rot="MR0">
 <attribute name="NAME" x="317.5" y="64.135" size="1.778" layer="95" rot="MR0"/>
 </instance>
@@
 <instance part="P+15" gate="1" x="76.2" y="43.18" rot="R90"/>
 <instance part="GND28" gate="1" x="73.66" y="38.1" rot="R270"/>
-<instance part="UPL" gate="A" x="264.16" y="63.5" rot="MR0"/>
-<instance part="UPL" gate="P" x="264.16" y="63.5"/>
+<instance part="OPAMP" gate="A" x="264.16" y="63.5" rot="MR0"/>
+<instance part="OPAMP" gate="P" x="264.16" y="63.5"/>
 <instance part="GND29" gate="1" x="264.16" y="50.8"/>
 <instance part="P+16" gate="1" x="264.16" y="78.74"/>
@@
 </segment>
 <segment>
-<pinref part="UPL" gate="P" pin="V-"/>
+<pinref part="OPAMP" gate="P" pin="V-"/>
 <wire x1="264.16" y1="55.88" x2="264.16" y2="53.34" width="0.1524" layer="91"/>
 <pinref part="GND29" gate="1" pin="GND"/>
@@
 </segment>
 <segment>
-<pinref part="UPL" gate="P" pin="V+"/>
+<pinref part="OPAMP" gate="P" pin="V+"/>
 <wire x1="264.16" y1="71.12" x2="264.16" y2="73.66" width="0.1524" layer="91"/>
 <pinref part="P+16" gate="1" pin="VCC"/>
@@
 <net name="N$20" class="0">
 <segment>
-<pinref part="UPL" gate="B" pin="+IN"/>
+<pinref part="OPAMP" gate="B" pin="+IN"/>
 <wire x1="337.82" y1="63.5" x2="327.66" y2="63.5" width="0.1524" layer="91"/>
 <pinref part="UP_CAP1" gate="G$1" pin="2"/>
@@
 <segment>
 <pinref part="R2" gate="G$1" pin="A"/>
-<pinref part="UPL" gate="B" pin="OUT"/>
+<pinref part="OPAMP" gate="B" pin="OUT"/>
 <wire x1="294.64" y1="60.96" x2="307.34" y2="60.96" width="0.1524" layer="91"/>
 <pinref part="UP_CAP3" gate="G$1" pin="1"/>
@@
 <wire x1="307.34" y1="50.8" x2="307.34" y2="53.34" width="0.1524" layer="91"/>
 <junction x="299.72" y="50.8"/>
-<pinref part="UPL" gate="B" pin="-IN"/>
+<pinref part="OPAMP" gate="B" pin="-IN"/>
 <wire x1="330.2" y1="58.42" x2="327.66" y2="58.42" width="0.1524" layer="91"/>
 <wire x1="330.2" y1="50.8" x2="330.2" y2="58.42" width="0.1524" layer="91"/>
@@
 </segment>
 <segment>
-<pinref part="UPL" gate="A" pin="OUT"/>
+<pinref part="OPAMP" gate="A" pin="OUT"/>
 <wire x1="256.54" y1="63.5" x2="248.92" y2="63.5" width="0.1524" layer="91"/>
 <label x="248.92" y="63.5" size="1.778" layer="95" rot="R180" xref="yes"/>
@@
 <wire x1="279.4" y1="60.96" x2="276.86" y2="60.96" width="0.1524" layer="91"/>
 <wire x1="276.86" y1="60.96" x2="276.86" y2="55.88" width="0.1524" layer="91"/>
-<pinref part="UPL" gate="A" pin="-IN"/>
+<pinref part="OPAMP" gate="A" pin="-IN"/>
 <wire x1="276.86" y1="60.96" x2="271.78" y2="60.96" width="0.1524" layer="91"/>
 <junction x="276.86" y="60.96"/>
@@
 <pinref part="R1" gate="G$1" pin="S"/>
 <wire x1="274.32" y1="68.58" x2="274.32" y2="66.04" width="0.1524" layer="91"/>
-<pinref part="UPL" gate="A" pin="+IN"/>
+<pinref part="OPAMP" gate="A" pin="+IN"/>
 <wire x1="274.32" y1="66.04" x2="271.78" y2="66.04" width="0.1524" layer="91"/>
 </segment>
