File: core/pcb/rev1.0/apex-iii-core/apex-iii-core.brd (EAGLE design)
At the start: 99.1 x 49.5 mm, 68 parts

Commit message: core pcb
Parts:
- moved NTR2_DCPLG2 36.8 mm to (33.8, 2.29), turned to 90 degrees
- moved NTR2_DCPLG1 35.8 mm to (35.8, 2.29), turned to 90 degrees
- moved NTR2_RES4 26.6 mm to (27.2, 2.29), turned to 270 degrees
- moved JP5 26.1 mm to (36.3, 29.0)
- moved GPS_RES3 24.2 mm to (63.2, 31.8), turned to 270 degrees
- moved NTR2_RES3 23.2 mm to (24.9, 2.29), turned to 90 degrees
- moved NTR2_RES2 20.8 mm to (29.5, 2.29), turned to 90 degrees
- moved NTR2_RES1 19.9 mm to (31.8, 2.29), turned to 270 degrees
- moved GPS_RES2 19.7 mm to (61.0, 31.8), turned to 90 degrees
- moved GPS_DCPLG 18.4 mm to (56.6, 31.8), turned to 270 degrees
- moved GPS_RES1 16.9 mm to (58.7, 31.8), turned to 90 degrees
- moved INTERNAL_TEMP 13.5 mm to (32.5, 33.3), turned to 180 degrees
- moved I2C_RES1 13.2 mm to (34.0, 39.9), turned to 270 degrees
- moved I2C_RES2 12.0 mm to (31.0, 39.9), turned to 270 degrees
- moved 1WIRE 10.4 mm to (23.4, 36.6), turned to 180 degrees
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Routing:
- net GND: track 0.00 -> 95.8 mm, vias 0 -> 8
- net VBATT: track 0.00 -> 86.7 mm
- net VCC: track 0.00 -> 55.3 mm
- net N$12: track 0.00 -> 34.5 mm
- net RF_IN: track 0.00 -> 20.7 mm
- net N$6: track 0.00 -> 12.8 mm
- net N$13: track 0.00 -> 12.7 mm
- net N$5: track 0.00 -> 11.4 mm
- net N$1: track 0.00 -> 9.04 mm
- net BATT_READ: track 0.00 -> 6.99 mm
- net N$4: track 0.00 -> 3.59 mm
- net N$16: track 0.00 -> 2.29 mm
- net N$3: track 0.00 -> 2.11 mm
- net N$8: track 0.00 -> 2.11 mm
- added copper zone on layer 16, net GND
Other:
- board text added: "APEX"
- board text added: "CORE"
- board text added: "III"
- board text added: "POWER"
- board text added: "STATUS"

Commit message: continued with PCB + readme
Parts:
- moved GPS_RES2 2.50 mm to (63.2, 30.7)
- moved GPS_RES3 2.50 mm to (61.0, 30.7)
- moved GPS_DCPLG 1.02 mm to (56.6, 30.7)
- moved GPS_RES1 1.02 mm to (58.7, 30.7)
- turned I2C_RES1 to 90 degrees
- turned I2C_RES2 to 90 degrees
- turned STATUS_RES to 90 degrees
Routing:
- net GPS_TX: track 0.00 -> 20.8 mm
- net VCC: track 55.3 -> 70.0 mm
- net N$14: track 0.00 -> 12.2 mm
- net GND: track 95.8 -> 88.4 mm, vias 8 -> 10
- net N$13: track 12.7 -> 11.5 mm
- net N$8: track 2.11 -> 2.74 mm

Commit message: core pcb
Parts:
- moved STATUS_LED 25.8 mm to (81.3, 34.5), turned to 90 degrees
- moved STATUS_RES 24.3 mm to (81.3, 32.5), turned to 0 degrees
- moved MISO_RES 12.1 mm to (87.4, 29.2), turned to 270 degrees
- moved GPS_RES2 2.29 mm to (61.0, 30.7)
- moved GPS_RES3 2.29 mm to (63.2, 30.7)
- moved SD_DCPLG 2.29 mm to (81.3, 39.6), turned to 0 degrees
- moved C7 0.36 mm to (64.0, 39.9)
- moved NTR2_RES1 0.36 mm to (31.5, 2.54)
- moved NTR2_RES4 0.36 mm to (26.9, 2.54), turned to 90 degrees
- moved NTR2_RES2 0.36 mm to (29.2, 2.54), turned to 270 degrees
- moved NTR2_RES3 0.36 mm to (24.6, 2.54), turned to 270 degrees
- moved C6 0.36 mm to (62.0, 39.9)
- moved C8 0.36 mm to (59.9, 39.9)
- turned RESET to 0 degrees
Routing:
- net GPS_TX: track 20.8 -> 59.3 mm
- net BATT_READ: track 6.99 -> 40.7 mm, vias 0 -> 2
- net AVR_RESET: track 0.00 -> 33.4 mm
- net GPS_RX: track 0.00 -> 32.7 mm
- net MISO: track 0.00 -> 22.8 mm
- net DGTL9: track 0.00 -> 17.5 mm, vias 0 -> 1
- net MOSI: track 0.00 -> 16.9 mm
- net N$14: track 12.2 -> 17.9 mm
- net SCK: track 0.00 -> 3.60 mm
- net VCC: track 70.0 -> 73.2 mm
- net N$12: track 34.5 -> 36.0 mm
- net N$16: track 2.29 -> 3.07 mm
- net N$8: track 2.74 -> 2.11 mm
- net GND: track 88.4 -> 88.1 mm, vias 10 -> 50
- added copper zone on layer 1, net GND

Commit message: pcb mainly finished
Parts:
- OPAMP: value CA3240ED -> MAX4477
- moved JP6 44.3 mm to (64.4, 14.4), flipped to the bottom
- moved C1 1.52 mm to (89.9, 23.4)
- moved C3 1.52 mm to (89.9, 19.6)
- moved STATUS_LED 1.27 mm to (81.3, 35.8)
- moved TEMP_DCPLG 0.51 mm to (27.2, 39.6)
- moved UP_RES1 0.51 mm to (23.4, 39.6)
- moved UP_CAP3 0.51 mm to (27.2, 31.0)
- moved UP_RES2 0.51 mm to (23.4, 31.0)
- moved MISO_RES 0.25 mm to (87.1, 29.2)
- moved UP_CAP1 0.25 mm to (27.2, 33.8)
- moved UP_RES4 0.25 mm to (23.4, 33.8)
- moved 1WIRE 0.25 mm to (23.4, 36.8)
- moved UP_CAP4 0.25 mm to (27.2, 36.8)
- renumbered UPL to OPAMP
Routing:
- net VCC: track 73.2 -> 338.3 mm, vias 0 -> 2
- net TX_1: track 0.00 -> 130.7 mm, vias 0 -> 2
- net TEMPERATURE: track 0.00 -> 84.9 mm, vias 0 -> 2
- net UPLINK: track 0.00 -> 77.4 mm, vias 0 -> 2
- net I2C_SDA: track 0.00 -> 72.1 mm, vias 0 -> 2
- net NTR2_RSSI: track 0.00 -> 67.9 mm, vias 0 -> 1
- net GND: track 88.1 -> 152.1 mm, vias 50 -> 54
- net I2C_SCL: track 0.00 -> 63.0 mm, vias 0 -> 1
- net TX_0: track 0.00 -> 62.9 mm, vias 0 -> 2
- net NTR2_AF: track 0.00 -> 51.3 mm
- net NTR2_EN: track 0.00 -> 51.2 mm, vias 0 -> 2
- net SCK: track 3.60 -> 42.9 mm, vias 0 -> 2
- net N$23: track 0.00 -> 37.5 mm, vias 0 -> 2
- net N$22: track 0.00 -> 35.2 mm, vias 0 -> 2
- net N$10: track 0.00 -> 35.2 mm
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Other:
- board text added: "."
- board text added: "ANLG-1"
- board text added: "ANLG-2"
- board text added: "APEXIII"
- board text added: "AVR"
- board text added: "BATT"
- board text added: "DGTL"
- board text added: "EXT-TX"
- board text added: "FTDI"
- board text added: "GND"
- board text added: "GPS"
- board text added: "I2C"
- board text added: "ICSP"
- board text added: "MICRO SD"
- board text added: "NTR2"
- board text added: "OPAMP"
- board text added: "PATEL"
- board text added: "PRIYESH"
- board text added: "RST"
- board text added: "TEMP"
- board text added: "V+"
- board text added: "VREG"
- board text removed: "APEX"
- board text removed: "III"

Commit message: Core pcb finished
Routing:
- net VCC: track 338.3 -> 341.6 mm
- net ANLG3: track 27.8 -> 28.9 mm
Other:
- board text added: "+"
- board text added: "-"
- board text added: "2"
- board text added: "3"
- board text added: "6"
- board text added: "7"
- board text added: "9"
- board text added: "C"
- board text added: "CTS"
- board text added: "D"
- board text added: "DTR"
- board text added: "MISO"
- board text added: "MOSI"
- board text added: "RXI"
- board text added: "SCK"
- board text added: "T"
- board text added: "TXO"
- board text added: "VCC"
