File: core/pcb/rev1.0/apex-iii-core/apex-iii-core.brd (EAGLE design)
At the start: 99.1 x 49.5 mm, 68 parts

Commit message: setup module folders
Parts:
- NTR2_DCPLG2: value 100uF -> 47uF
Changed lines of the file:
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@@
 <element name="TEMP_DCPLG" library="SparkFun" package="0805" value="100nF" x="27.178" y="39.624" rot="R180"/>
 <element name="GPS_DCPLG" library="SparkFun" package="0805" value="100nF" x="56.642" y="30.734" rot="R270"/>
-<element name="NTR2_DCPLG2" library="SparkFun" package="0805" value="100uF" x="33.782" y="2.286" rot="R90"/>
+<element name="NTR2_DCPLG2" library="SparkFun" package="0805" value="47uF" x="33.782" y="2.286" rot="R90"/>
 <element name="SD_DCPLG" library="SparkFun" package="0805" value="100nF" x="81.28" y="39.624"/>
 <element name="VREG" library="linear-technology" package="SOIC8" value="LT1763CS8-3.3" x="93.98" y="14.224" rot="R270">
@@
 </signal>
 </signals>
-<errors>
-</errors>
 </board>
 </drawing>
