File: modules/adc_lemon/pcb/rev1.0/adc_lemon.brd (EAGLE design)
At the start: 40.1 x 31.7 mm, 24 parts, among them IC1 PICAXE-08M2, IC2 PICAXE-08M2

Commit message: fix airwires, rename, export larger pngs
Changed lines of the file:
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@@
 <wire x1="33.702" y1="9.064" x2="33.702" y2="9.798" width="0.254" layer="1"/>
 <wire x1="33.702" y1="9.798" x2="29.972" y2="13.528" width="0.254" layer="1"/>
-<polygon width="0.254" layer="16" isolate="0.254">
-<vertex x="-1.27" y="31.75"/>
-<vertex x="-1.27" y="32.512"/>
-<vertex x="0.254" y="34.036"/>
-<vertex x="39.878" y="34.036"/>
-<vertex x="42.164" y="31.75"/>
-<vertex x="42.164" y="-0.254"/>
-<vertex x="39.116" y="-3.302"/>
-<vertex x="-2.794" y="-3.302"/>
-<vertex x="-3.81" y="-2.286"/>
-<vertex x="-3.81" y="29.21"/>
-</polygon>
 <wire x1="19.732" y1="9.064" x2="19.732" y2="13.194" width="0.254" layer="1"/>
 <wire x1="19.732" y1="13.194" x2="20.066" y2="13.528" width="0.254" layer="1"/>
@@
 <via x="6.096" y="1.016" extent="1-16" drill="0.508"/>
 <wire x1="6.096" y1="1.016" x2="6.35" y2="1.016" width="0.254" layer="16"/>
+<polygon width="0.254" layer="16" isolate="0.254">
+<vertex x="0" y="0"/>
+<vertex x="40.132" y="0"/>
+<vertex x="40.132" y="31.75"/>
+<vertex x="0" y="31.75"/>
+</polygon>
 </signal>
 <signal name="SCL">
